Commit message: joint state working

File: one_joint.urdf (robot description, URDF)
Before this commit: robot one_joint_robot, 2 links, 1 joints
Links:
- link base_link: geometry 
- link link1: geometry 
Joints:
- joint joint1: limit (none) -> lower=-6.28 upper=6.28 effort=10 velocity=5; origin xyz=0 0 0.05 -> xyz=0 0 0 rpy=0 0 0; type continuous -> revolute
